File: KiCad/SCH1110-2 - IO Module PCB/SCH1110 - IO Module PCB.kicad_pcb (KiCad board)
At the start: 2 copper layers, 60.3 x 50.8 mm, 33 parts, among them J1 Radio In, J2 3.5mm Audio In, J3 Power/Input Switch, J4 Power In, J5 Headset Out, K1 TXS2, U1 5532, U2 MAX4466, U3 uA78M05

Commit message: Review changes and adjustments
Parts:
- moved J4 0.38 mm to (105.3, 85.0), turned to 270 degrees
Connections:
- J4 pad 1: +9V -> Earth
- J4 pad 2: Earth -> +9V
Routing:
- net /AUDIO_SELECT: track 11.9 -> 12.8 mm
- net Earth: track 39.6 -> 40.5 mm
Changed lines of the file:
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@@
     (thickness 1.6)
     (drawings 18)
-    (tracks 269)
+    (tracks 272)
     (zones 0)
     (modules 33)
@@
   )
   (setup
-    (last_trace_width 0.254)
+    (last_trace_width 0.381)
     (user_trace_width 0.381)
     (user_trace_width 0.508)
@@
     (aux_axis_origin 0 0)
     (grid_origin 101.6 101.6)
-    (visible_elements FFFFFF7F)
+    (visible_elements 7FFFFFFF)
     (pcbplotparams
       (layerselection 0x010fc_ffffffff)
-      (usegerberextensions false)
+      (usegerberextensions true)
       (usegerberattributes false)
       (usegerberadvancedattributes false)
@@
       (outputformat 1)
       (mirror false)
-      (drillshape 1)
+      (drillshape 0)
       (scaleselection 1)
-      (outputdirectory ""))
+      (outputdirectory "Gerbers/"))
   )
   (net 0 "")
@@
     (add_net "Net-(R8-Pad1)")
     (add_net PTT)
+  )
+  (module conn-wire-pads:WP-75mil-1x02 (layer F.Cu)
+    (at 105.283 84.963 270)
+    (descr "Wire pads - 75mil x 150 mil - Single row, 2 pos.")
+    (attr virtual)
+    (fp_text reference J4 (at -3.81 -3.175 270) (layer F.SilkS)
+      (effects (font (size 1 1) (thickness 0.18)) (justify left bottom))
+    )
+    (fp_text value "Power In" (at 0 3.81 270) (layer F.Fab) hide
+      (effects (font (size 1 1) (thickness 0.18)))
+    )
+    (fp_line (start -3.81 2.54) (end -3.81 -2.54) (layer F.CrtYd) (width 0.05))
+    (fp_line (start 3.81 2.54) (end -3.81 2.54) (layer F.CrtYd) (width 0.05))
+    (fp_line (start 3.81 -2.54) (end 3.81 2.54) (layer F.CrtYd) (width 0.05))
+    (fp_line (start -3.81 -2.54) (end 3.81 -2.54) (layer F.CrtYd) (width 0.05))
+    (fp_line (start -3.81 2.54) (end -3.81 -2.54) (layer F.SilkS) (width 0.18))
+    (fp_line (start 3.81 2.54) (end -3.81 2.54) (layer F.SilkS) (width 0.18))
+    (fp_line (start 3.81 -2.54) (end 3.81 2.54) (layer F.SilkS) (width 0.18))
+    (fp_line (start -3.81 -2.54) (end 3.81 -2.54) (layer F.SilkS) (width 0.18))
+    (pad 2 smd oval (at 1.905 0 270) (size 1.905 3.81) (layers F.Cu F.Paste F.Mask)
+      (net 8 +9V))
+    (pad 1 smd oval (at -1.905 0 270) (size 1.905 3.81) (layers F.Cu F.Paste F.Mask)
+      (net 5 Earth))
   )
   (module digikey-footprints:0805 (layer F.Cu)
@@
       (net 16 /AUDIO_SELECT))
   )
-  (module conn-wire-pads:WP-75mil-1x02 (layer F.Cu)
-    (at 105.283 84.582 90)
-    (descr "Wire pads - 75mil x 150 mil - Single row, 2 pos.")
-    (attr virtual)
-    (fp_text reference J4 (at -5.461 -1.016 180) (layer F.SilkS)
-      (effects (font (size 1 1) (thickness 0.18)) (justify left bottom))
-    )
-    (fp_text value "Power In" (at 0 3.81 90) (layer F.Fab) hide
-      (effects (font (size 1 1) (thickness 0.18)))
-    )
-    (fp_line (start -3.81 2.54) (end -3.81 -2.54) (layer F.CrtYd) (width 0.05))
-    (fp_line (start 3.81 2.54) (end -3.81 2.54) (layer F.CrtYd) (width 0.05))
-    (fp_line (start 3.81 -2.54) (end 3.81 2.54) (layer F.CrtYd) (width 0.05))
-    (fp_line (start -3.81 -2.54) (end 3.81 -2.54) (layer F.CrtYd) (width 0.05))
-    (fp_line (start -3.81 2.54) (end -3.81 -2.54) (layer F.SilkS) (width 0.18))
-    (fp_line (start 3.81 2.54) (end -3.81 2.54) (layer F.SilkS) (width 0.18))
-    (fp_line (start 3.81 -2.54) (end 3.81 2.54) (layer F.SilkS) (width 0.18))
-    (fp_line (start -3.81 -2.54) (end 3.81 -2.54) (layer F.SilkS) (width 0.18))
-    (pad 2 smd oval (at 1.905 0 90) (size 1.905 3.81) (layers F.Cu F.Paste F.Mask)
-      (net 5 Earth))
-    (pad 1 smd oval (at -1.905 0 90) (size 1.905 3.81) (layers F.Cu F.Paste F.Mask)
-      (net 8 +9V))
-  )
   (module conn-wire-pads:WP-75mil-1x04 (layer F.Cu)
     (at 109.855 56.261 180)
@@
   (segment (start 113.157 71.917) (end 113.573 71.501) (width 0.381) (layer F.Cu) (net 5))
   (segment (start 113.157 72.279) (end 113.157 71.917) (width 0.381) (layer F.Cu) (net 5))
-  (segment (start 108.1615 84.603) (end 109.876 84.603) (width 0.381) (layer F.Cu) (net 5))
-  (segment (start 105.283 82.677) (end 106.2355 82.677) (width 0.381) (layer F.Cu) (net 5))
-  (segment (start 106.2355 82.677) (end 108.1615 84.603) (width 0.381) (layer F.Cu) (net 5))
   (segment (start 111.332 84.603) (end 115.676 84.603) (width 0.381) (layer F.Cu) (net 5))
   (segment (start 109.876 84.603) (end 111.332 84.603) (width 0.381) (layer F.Cu) (net 5))
@@
   (via (at 109.876 81.767) (size 0.762) (drill 0.381) (layers F.Cu B.Cu) (net 5))
   (segment (start 109.876 84.603) (end 109.876 81.767) (width 0.508) (layer F.Cu) (net 5))
-  (segment (start 105.283 82.677) (end 105.283 80.645) (width 0.508) (layer F.Cu) (net 5))
-  (via (at 105.283 80.645) (size 0.762) (drill 0.381) (layers F.Cu B.Cu) (net 5))
   (via (at 117.856 75.311) (size 0.762) (drill 0.381) (layers F.Cu B.Cu) (net 5))
   (segment (start 116.459 75.119) (end 117.664 75.119) (width 0.381) (layer F.Cu) (net 5))
@@
   (segment (start 130.265 86.143) (end 130.4925 85.9155) (width 0.381) (layer F.Cu) (net 5))
   (segment (start 130.4925 85.9155) (end 130.6195 85.7885) (width 0.381) (layer F.Cu) (net 5))
+  (segment (start 107.569 83.058) (end 108.204 83.693) (width 0.381) (layer F.Cu) (net 5))
+  (segment (start 105.283 83.058) (end 107.569 83.058) (width 0.381) (layer F.Cu) (net 5))
+  (segment (start 108.42 84.603) (end 109.876 84.603) (width 0.381) (layer F.Cu) (net 5))
+  (segment (start 108.204 84.387) (end 108.42 84.603) (width 0.381) (layer F.Cu) (net 5))
+  (segment (start 108.204 83.693) (end 108.204 84.387) (width 0.381) (layer F.Cu) (net 5))
+  (via (at 105.283 80.391) (size 0.762) (drill 0.381) (layers F.Cu B.Cu) (net 5))
+  (segment (start 105.283 83.058) (end 105.283 80.391) (width 0.381) (layer F.Cu) (net 5))
   (segment (start 110.109 75.181) (end 110.109 73.725) (width 0.254) (layer F.Cu) (net 6))
   (segment (start 112.589 73.725) (end 112.668 73.646) (width 0.254) (layer F.Cu) (net 6))
@@
   (segment (start 121.539 86.487) (end 121.539 87.376) (width 0.254) (layer F.Cu) (net 7))
   (segment (start 121.539 87.376) (end 121.985 87.822) (width 0.254) (layer F.Cu) (net 7))
-  (segment (start 107.569 86.487) (end 108.585 87.503) (width 0.381) (layer F.Cu) (net 8))
-  (segment (start 105.283 86.487) (end 107.569 86.487) (width 0.381) (layer F.Cu) (net 8))
-  (segment (start 108.585 87.503) (end 111.379 87.503) (width 0.381) (layer F.Cu) (net 8))
-  (segment (start 111.979 86.903) (end 115.676 86.903) (width 0.381) (layer F.Cu) (net 8))
-  (segment (start 111.379 87.503) (end 111.979 86.903) (width 0.381) (layer F.Cu) (net 8))
   (segment (start 124.646 81.243) (end 125.349 81.243) (width 0.381) (layer F.Cu) (net 8))
   (segment (start 123.063 82.045) (end 123.844 82.045) (width 0.381) (layer F.Cu) (net 8))
@@
   (segment (start 122.171 82.045) (end 123.063 82.045) (width 0.381) (layer F.Cu) (net 8))
   (segment (start 121.539 82.677) (end 122.171 82.045) (width 0.381) (layer F.Cu) (net 8))
+  (segment (start 114.011 86.903) (end 115.676 86.903) (width 0.381) (layer F.Cu) (net 8))
+  (segment (start 113.538 87.376) (end 114.011 86.903) (width 0.381) (layer F.Cu) (net 8))
+  (segment (start 108.458 87.376) (end 113.538 87.376) (width 0.381) (layer F.Cu) (net 8))
+  (segment (start 105.283 86.868) (end 107.95 86.868) (width 0.381) (layer F.Cu) (net 8))
+  (segment (start 107.95 86.868) (end 108.458 87.376) (width 0.381) (layer F.Cu) (net 8))
   (segment (start 114.741 76.519) (end 114.568 76.346) (width 0.381) (layer F.Cu) (net 9))
   (segment (start 116.459 76.519) (end 114.741 76.519) (width 0.381) (layer F.Cu) (net 9))
@@
   (segment (start 139.319 64.897) (end 139.319 67.691) (width 0.381) (layer F.Cu) (net 16))
   (segment (start 140.081 64.135) (end 139.319 64.897) (width 0.381) (layer F.Cu) (net 16))
+  (segment (start 140.081 56.134) (end 140.081 55.1815) (width 0.508) (layer F.Cu) (net 16))
   (segment (start 111.76 55.3085) (end 111.76 56.261) (width 0.254) (layer F.Cu) (net 17))
   (segment (start 120.901 56.769) (end 119.888 56.769) (width 0.254) (layer F.Cu) (net 17))
@@
   (segment (start 126.619 86.143) (end 126.619 89.219) (width 0.254) (layer F.Cu) (net 22))
   (segment (start 126.557 89.281) (end 127.886 89.281) (width 0.254) (layer F.Cu) (net 22))
+  (segment (start 126.489 81.113) (end 126.619 81.243) (width 0.254) (layer F.Cu) (net 23))
+  (segment (start 126.489 79.121) (end 126.489 81.113) (width 0.254) (layer F.Cu) (net 23))
+  (segment (start 123.063 83.374) (end 126.176 83.374) (width 0.254) (layer F.Cu) (net 23))
+  (segment (start 126.619 82.931) (end 126.619 81.243) (width 0.254) (layer F.Cu) (net 23))
+  (segment (start 126.176 83.374) (end 126.619 82.931) (width 0.254) (layer F.Cu) (net 23))
+  (segment (start 127.889 79.121) (end 127.889 81.243) (width 0.254) (layer F.Cu) (net 24))
   (segment (start 130.664 80.518) (end 129.921 81.261) (width 0.254) (layer F.Cu) (net 25))
   (segment (start 131.318 80.518) (end 130.664 80.518) (width 0.254) (layer F.Cu) (net 25))
@@
   (segment (start 128.443 77.343) (end 129.159 78.059) (width 0.254) (layer F.Cu) (net 25))
   (segment (start 127.889 77.343) (end 128.443 77.343) (width 0.254) (layer F.Cu) (net 25))
-  (segment (start 126.489 81.113) (end 126.619 81.243) (width 0.254) (layer F.Cu) (net 23))
-  (segment (start 126.489 79.121) (end 126.489 81.113) (width 0.254) (layer F.Cu) (net 23))
-  (segment (start 123.063 83.374) (end 126.176 83.374) (width 0.254) (layer F.Cu) (net 23))
-  (segment (start 126.619 82.931) (end 126.619 81.243) (width 0.254) (layer F.Cu) (net 23))
-  (segment (start 126.176 83.374) (end 126.619 82.931) (width 0.254) (layer F.Cu) (net 23))
-  (segment (start 127.889 79.121) (end 127.889 81.243) (width 0.254) (layer F.Cu) (net 24))
   (segment (start 127.889 70.104) (end 127.889 77.343) (width 0.254) (layer F.Cu) (net 25))
   (segment (start 129.54 64.008) (end 129.54 68.453) (width 0.254) (layer F.Cu) (net 25))
