File: KiCad/SCH1110-2 - IO Module PCB/SCH1110 - IO Module PCB.sch (KiCad schematic (older format))
At the start: 33 parts, among them J1 Radio In, J2 3.5mm Audio In, J3 Power/Input Switch, J4 Power In, J5 Headset Out, K1 TXS2, U1 5532, U2 MAX4466, U3 uA78M05

Commit message: Review changes and adjustments
Parts:
- removed J4: Power In, conn-wire-pads:WP-75mil-1x02, symbol Connector:Conn_01x02_Female
- added J4: Power In, conn-wire-pads:WP-75mil-1x02, symbol SCH1110---IO-Module-PCB-rescue:Conn_01x02_Female-Connector
- C1, C10, C9: symbol Device:CP1 -> SCH1110---IO-Module-PCB-rescue:CP1-Device
- C11, C2, C3, C4, C5, C6, C7, C8: symbol Device:C -> SCH1110---IO-Module-PCB-rescue:C-Device
- J1, J2, J3: symbol Connector:Conn_01x02_Female -> SCH1110---IO-Module-PCB-rescue:Conn_01x02_Female-Connector
- J5: symbol Connector:Conn_01x04_Female -> SCH1110---IO-Module-PCB-rescue:Conn_01x04_Female-Connector
- R1, R10, R11, R12, R2, R3, R4, R5, R6, R7, R8, R9: symbol Device:R -> SCH1110---IO-Module-PCB-rescue:R-Device
- RV1: symbol Device:R_POT_TRIM -> SCH1110---IO-Module-PCB-rescue:R_POT_TRIM-Device
Connections:
- net +9V: now also J4.2 (Pin_2)
- net Earth: now also J4.1 (Pin_1)
Changed lines of the file:
@@
 $EndDescr
 $Comp
-L Device:R R1
+L SCH1110---IO-Module-PCB-rescue:R-Device R1
 U 1 1 5B749509
 P 2000 5700
@@
 Wire Wire Line
 	9150 3700 9150 3950
-Text Label 8950 3950 2    50   ~ 0
-AUDIO_SELECT
 Text Label 9750 5200 2    50   ~ 0
 R_CH_OUT
@@
 L_CH_OUT
 $Comp
-L Connector:Conn_01x02_Female J3
+L SCH1110---IO-Module-PCB-rescue:Conn_01x02_Female-Connector J3
 U 1 1 5C673D07
 P 9250 3500
@@
 $EndComp
 $Comp
-L Connector:Conn_01x02_Female J2
+L SCH1110---IO-Module-PCB-rescue:Conn_01x02_Female-Connector J2
 U 1 1 5C6744BE
 P 7600 3500
@@
 $EndComp
 $Comp
-L Connector:Conn_01x04_Female J5
+L SCH1110---IO-Module-PCB-rescue:Conn_01x04_Female-Connector J5
 U 1 1 5C674628
 P 10150 3500
@@
 $EndComp
 $Comp
-L power:Earth #PWR07
+L SCH1110---IO-Module-PCB-rescue:Earth-power #PWR07
 U 1 1 5CAB1C0E
 P 3850 5600
@@
 	9250 3700 9250 4800
 $Comp
-L power:+5V #PWR03
+L SCH1110---IO-Module-PCB-rescue:+5V-power #PWR03
 U 1 1 5CABA565
 P 2800 4450
@@
 $EndComp
 $Comp
-L Device:C C2
+L SCH1110---IO-Module-PCB-rescue:C-Device C2
 U 1 1 5CABBD0C
 P 2400 5400
@@
 	3500 5300 3250 5300
 $Comp
-L Device:C C4
+L SCH1110---IO-Module-PCB-rescue:C-Device C4
 U 1 1 5CAC002E
 P 3800 6550
@@
 $EndComp
 $Comp
-L Device:R R7
+L SCH1110---IO-Module-PCB-rescue:R-Device R7
 U 1 1 5CAC0652
 P 3550 6000
@@
 $EndComp
 $Comp
-L Device:R R6
+L SCH1110---IO-Module-PCB-rescue:R-Device R6
 U 1 1 5CAC0C51
 P 3250 6850
@@
 	3650 6550 3250 6550
 $Comp
-L Device:C C3
+L SCH1110---IO-Module-PCB-rescue:C-Device C3
 U 1 1 5CAC865D
 P 3250 7250
@@
 	3250 7000 3250 7100
 $Comp
-L power:Earth #PWR05
+L SCH1110---IO-Module-PCB-rescue:Earth-power #PWR05
 U 1 1 5CACD96C
 P 3250 7500
@@
 	3250 7500 3250 7400
 $Comp
-L Device:R R4
+L SCH1110---IO-Module-PCB-rescue:R-Device R4
 U 1 1 5CACF5BA
 P 2800 4750
@@
 $EndComp
 $Comp
-L Device:R R5
+L SCH1110---IO-Module-PCB-rescue:R-Device R5
 U 1 1 5CACFF5C
 P 2800 5450
@@
 $EndComp
 $Comp
-L power:Earth #PWR04
+L SCH1110---IO-Module-PCB-rescue:Earth-power #PWR04
 U 1 1 5CAD2E89
 P 2800 5700
@@
 	2800 5600 2800 5700
 $Comp
-L power:+5V #PWR06
+L SCH1110---IO-Module-PCB-rescue:+5V-power #PWR06
 U 1 1 5CAD389A
 P 3850 4800
@@
 	2400 5100 2800 5100
 $Comp
-L Device:R R9
+L SCH1110---IO-Module-PCB-rescue:R-Device R9
 U 1 1 5CAEDA29
 P 5050 5200
@@
 $EndComp
 $Comp
-L Device:R R8
+L SCH1110---IO-Module-PCB-rescue:R-Device R8
 U 1 1 5CAEE66F
 P 5050 4750
@@
 $EndComp
 $Comp
-L Device:R R11
+L SCH1110---IO-Module-PCB-rescue:R-Device R11
 U 1 1 5CB04BC4
 P 5800 5750
@@
 Connection ~ 5350 5200
 $Comp
-L Device:R R10
+L SCH1110---IO-Module-PCB-rescue:R-Device R10
 U 1 1 5CB0A8C3
 P 5350 6050
@@
 $EndComp
 $Comp
-L power:Earth #PWR011
+L SCH1110---IO-Module-PCB-rescue:Earth-power #PWR011
 U 1 1 5CB0FBF4
 P 5350 6750
@@
 	4550 5200 4250 5200
 $Comp
-L Device:R R2
+L SCH1110---IO-Module-PCB-rescue:R-Device R2
 U 1 1 5CB3A93B
 P 3250 3300
@@
 $EndComp
 $Comp
-L Device:R R3
+L SCH1110---IO-Module-PCB-rescue:R-Device R3
 U 1 1 5CB3FBC0
 P 3250 3850
@@
 $EndComp
 $Comp
-L Device:C C6
+L SCH1110---IO-Module-PCB-rescue:C-Device C6
 U 1 1 5CB5BBBA
 P 5700 1900
@@
 $EndComp
 $Comp
-L power:Earth #PWR09
+L SCH1110---IO-Module-PCB-rescue:Earth-power #PWR09
 U 1 1 5CB5E74D
 P 5100 2300
@@
 	5100 1950 5100 2150
 $Comp
-L Device:C C5
+L SCH1110---IO-Module-PCB-rescue:C-Device C5
 U 1 1 5CB6F7D1
 P 4550 1900
@@
 	5700 2150 5100 2150
 $Comp
-L power:+5V #PWR012
+L SCH1110---IO-Module-PCB-rescue:+5V-power #PWR012
 U 1 1 5CB78869
 P 7400 1400
@@
 $EndComp
 $Comp
-L power:+9V #PWR014
+L SCH1110---IO-Module-PCB-rescue:+9V-power #PWR014
 U 1 1 5CB788DD
 P 8250 1400
@@
 $EndComp
 $Comp
-L Device:C C7
+L SCH1110---IO-Module-PCB-rescue:C-Device C7
 U 1 1 5CB78A4C
 P 7400 1700
@@
 $EndComp
 $Comp
-L Device:C C8
+L SCH1110---IO-Module-PCB-rescue:C-Device C8
 U 1 1 5CB7B05D
 P 8250 1700
@@
 $EndComp
 $Comp
-L power:Earth #PWR013
+L SCH1110---IO-Module-PCB-rescue:Earth-power #PWR013
 U 1 1 5CB7D71C
 P 7400 2000
@@
 $EndComp
 $Comp
-L power:Earth #PWR015
+L SCH1110---IO-Module-PCB-rescue:Earth-power #PWR015
 U 1 1 5CB7FD1D
 P 8250 2000
@@
 Place close to U2
 $Comp
-L power:+5V #PWR010
+L SCH1110---IO-Module-PCB-rescue:+5V-power #PWR010
 U 1 1 5CB9BD33
 P 5700 1450
@@
 	5700 1450 5700 1600
 $Comp
-L power:+9V #PWR08
+L SCH1110---IO-Module-PCB-rescue:+9V-power #PWR08
 U 1 1 5CB9E7B8
 P 4550 1450
@@
 	4550 1450 4550 1600
 $Comp
-L power:+9V #PWR01
+L SCH1110---IO-Module-PCB-rescue:+9V-power #PWR01
 U 1 1 5CBA12F3
 P 4000 3050
@@
 $EndComp
 $Comp
-L power:Earth #PWR02
+L SCH1110---IO-Module-PCB-rescue:Earth-power #PWR02
 U 1 1 5CBA3F4A
 P 3250 4400
@@
 	3250 4250 3250 4400
 $Comp
-L Connector:Conn_01x02_Female J4
-U 1 1 5CBA9D97
-P 9700 950
-F 0 "J4" V 9640 762 50  0000 R CNN
-F 1 "Power In" V 9800 1200 50  0000 R CNN
-F 2 "conn-wire-pads:WP-75mil-1x02" H 9700 950 50  0001 C CNN
-F 3 "~" H 9700 950 50  0001 C CNN
-	1    9700 950
-	0    -1   -1   0
-$EndComp
-$Comp
-L power:+9V #PWR016
+L SCH1110---IO-Module-PCB-rescue:+9V-power #PWR016
 U 1 1 5CBACC7F
-P 9200 1150
-F 0 "#PWR016" H 9200 1000 50  0001 C CNN
-F 1 "+9V" H 9215 1323 50  0000 C CNN
-F 2 "" H 9200 1150 50  0001 C CNN
-F 3 "" H 9200 1150 50  0001 C CNN
-	1    9200 1150
-	1    0    0    -1
-$EndComp
-$Comp
-L power:Earth #PWR017
-U 1 1 5CBBDF98
-P 9800 1450
-F 0 "#PWR017" H 9800 1200 50  0001 C CNN
-F 1 "Earth" H 9800 1300 50  0001 C CNN
-F 2 "" H 9800 1450 50  0001 C CNN
-F 3 "~" H 9800 1450 50  0001 C CNN
-	1    9800 1450
-	1    0    0    -1
-$EndComp
-Wire Wire Line
-	9200 1150 9200 1350
-Wire Wire Line
-	9200 1350 9700 1350
-Wire Wire Line
-	9700 1350 9700 1150
-Wire Wire Line
-	9800 1150 9800 1450
+P 9150 1100
+F 0 "#PWR016" H 9150 950 50  0001 C CNN
+F 1 "+9V" H 9165 1273 50  0000 C CNN
+F 2 "" H 9150 1100 50  0001 C CNN
+F 3 "" H 9150 1100 50  0001 C CNN
+	1    9150 1100
+	1    0    0    -1
+$EndComp
 Wire Wire Line
 	5350 5750 5350 5900
@@
 Connection ~ 3250 6000
 $Comp
-L Device:R_POT_TRIM RV1
+L SCH1110---IO-Module-PCB-rescue:R_POT_TRIM-Device RV1
 U 1 1 5CB65E6D
 P 4150 6000
@@
 	2000 2600 2000 5350
 $Comp
-L Connector:Conn_01x02_Female J1
+L SCH1110---IO-Module-PCB-rescue:Conn_01x02_Female-Connector J1
 U 1 1 5C67457B
 P 2100 2400
@@
 $EndComp
 $Comp
-L Device:R R12
+L SCH1110---IO-Module-PCB-rescue:R-Device R12
 U 1 1 5CB7B538
 P 4200 4100
@@
 	4550 4750 4900 4750
 $Comp
-L power:+5V #PWR0101
+L SCH1110---IO-Module-PCB-rescue:+5V-power #PWR0101
 U 1 1 5CC0B8C8
 P 3250 2750
@@
 	3250 2750 3250 3150
 $Comp
-L Device:C C11
+L SCH1110---IO-Module-PCB-rescue:C-Device C11
 U 1 1 5CC13127
 P 5350 6450
@@
 	5350 6600 5350 6750
 $Comp
-L Device:CP1 C10
+L SCH1110---IO-Module-PCB-rescue:CP1-Device C10
 U 1 1 5CC1A748
 P 3000 3550
@@
 $EndComp
 $Comp
-L Device:CP1 C9
+L SCH1110---IO-Module-PCB-rescue:CP1-Device C9
 U 1 1 5CC2CF65
 P 6750 5300
@@
 $EndComp
 $Comp
-L Device:CP1 C1
+L SCH1110---IO-Module-PCB-rescue:CP1-Device C1
 U 1 1 5CC38145
 P 1650 5650
@@
 	-1   0    0    1
 $EndComp
+$Comp
+L SCH1110---IO-Module-PCB-rescue:Conn_01x02_Female-Connector J4
+U 1 1 5CB32E57
+P 9950 1000
+F 0 "J4" V 9890 812 50  0000 R CNN
+F 1 "Power In" V 10050 1100 50  0000 R CNN
+F 2 "conn-wire-pads:WP-75mil-1x02" H 9950 1000 50  0001 C CNN
+F 3 "~" H 9950 1000 50  0001 C CNN
+	1    9950 1000
+	0    1    -1   0
+$EndComp
+$Comp
+L SCH1110---IO-Module-PCB-rescue:Earth-power #PWR0102
+U 1 1 5CB3A0E6
+P 9950 1600
+F 0 "#PWR0102" H 9950 1350 50  0001 C CNN
+F 1 "Earth" H 9950 1450 50  0001 C CNN
+F 2 "" H 9950 1600 50  0001 C CNN
+F 3 "~" H 9950 1600 50  0001 C CNN
+	1    9950 1600
+	1    0    0    -1
+$EndComp
+Wire Wire Line
+	9950 1200 9950 1600
+Wire Wire Line
+	9850 1200 9850 1400
+Wire Wire Line
+	9850 1400 9150 1400
+Wire Wire Line
+	9150 1100 9150 1400
+Text Label 8500 3950 0    50   ~ 0
+AUDIO_SELECT
 $EndSCHEMATC
